File: danger.brd (EAGLE design)
At the start: 160 x 134.3 mm, 7 parts

Commit message: redid based on sparkfun design
Parts:
- removed U$1, U$3: SLIDER, SparkFun-Electromechanical:SLIDER
- removed U$4: SPARK_CORE, Spark:SPARK_CORE_STACKABLE
- added C1, C2: 0.1uF, SparkFun-Passives:CAP-PTH-SMALL2
- added C3: 10pF, SparkFun-Passives:CAP-PTH-SMALL2
- added IC1: SPARK_CORECORE, Spark:SPARK_CORE
- added JP1: (no value), SparkFun:1X05
- added LED1: Red, SparkFun:LED5MM
- added LED2: Yellow, SparkFun:LED5MM
- added LED3: Green, SparkFun:LED5MM
- added R1, R10, R11, R12, R13, R14, R15, R16, R2, R3, R9: 330, SparkFun:AXIAL-0.3
- added R17: 1k, SparkFun:AXIAL-0.3
- added R30: 10K, SparkFun:AXIAL-0.3
- added R4: 10M, SparkFun:AXIAL-0.3
- added R5: CdS, SparkFun:PHOTOCELL
- added R6: Slider3, SparkFun:SLIDER
- added R7: Slider2, SparkFun:SLIDER
- added R8: Slider1, SparkFun:SLIDER
- added SG1: BUZZER, SparkFun:BUZZER-12MM
- added U2: 74LS595N, SparkFun:DIL16
- added U4: TMP36, SparkFun-Sensors:TO-92
- added U6: 7-SEGMENT-DISPLAY-1"-RED, SparkFun:7-SEGMENT-1"PTH
- S1: value (none) -> Button1; device SparkFun-Electromechanical:TACTILE-PTH -> SparkFun:TACTILE-PTH-12MM
- S2: value (none) -> Button2; device SparkFun-Electromechanical:TACTILE-PTH -> SparkFun:TACTILE-PTH-12MM
- S3: value (none) -> Button3; device SparkFun-Electromechanical:TACTILE-PTH -> SparkFun:TACTILE-PTH-12MM
- U$2: value SLIDER -> OSHW-LOGOM; device SparkFun-Electromechanical:SLIDER -> SparkFun-Aesthetics:OSHW-LOGO-M
- moved S3 82.8 mm to (59.7, 10.2)
- moved S2 58.8 mm to (44.5, 10.2)
- moved U$2 58.7 mm to (80.0, 10.2), turned to 0 degrees
- moved S1 34.9 mm to (29.2, 10.2)
Connections:
- removed net RAW: U$4.#1, U$4.1, U$4.@1
- new net B1: IC1.13, S1.3
- new net B2: IC1.14, S2.3
- new net B3: IC1.15, S3.3
- new net BUZZER: IC1.3, SG1.+
- new net CDS: IC1.6, R30.P$2, R5.1
- new net CLOCK: IC1.9, JP1.3, U2.11
- new net LATCH: IC1.8, JP1.2, U2.12
- new net LED_G: IC1.20, LED3.A
- new net LED_R: IC1.18, LED1.A
- new net LED_Y: IC1.19, LED2.A
- new net N$10: R16.P$1, U2.7
- new net N$11: R9.P$2, U6.7
- new net N$12: R10.P$2, U6.6
- new net N$13: R11.P$2, U6.4
- new net N$14: R12.P$2, U6.2
- new net N$15: R13.P$2, U6.1
- new net N$16: R14.P$2, U6.9
- new net N$17: R15.P$2, U6.10
- new net N$18: R16.P$2, U6.5
- new net N$19: LED2.K, R2.P$2
- new net N$2: R9.P$1, U2.15
- new net N$20: LED3.K, R3.P$2
- new net N$3: LED1.K, R1.P$2
- new net N$4: R10.P$1, U2.1
- new net N$5: R11.P$1, U2.2
- new net N$6: R12.P$1, U2.3
- new net N$7: R13.P$1, U2.4
- new net N$8: R14.P$1, U2.5
- new net N$9: R15.P$1, U2.6
- new net S1: IC1.12, R8.2A
- new net S2: IC1.11, R7.2A
- new net S3: IC1.10, R6.2A
- new net SERIAL_IN: IC1.7, U2.14
- new net SERIAL_OUT: JP1.4, U2.9
- new net TEMP: IC1.5, U4.2
- new net TOUCH: C3.1, R17.P$2, R4.P$2
- new net TOUCH_R: IC1.16, R17.P$1
- new net TOUCH_S: IC1.17, R4.P$1
- net GND: now also C1.2, C2.2, C3.2, IC1.2, IC1.21, JP1.5, R1.P$1, R2.P$1, R3.P$1, R30.P$1, R6.3, R7.3, R8.3, S1.1, S2.1, S3.1, SG1.-, U2.13, U2.8, U4.3; no longer U$4.#2, U$4.#21, U$4.2, U$4.21, U$4.@2, U$4.@21
- net VCC: now also C1.1, C2.1, IC1.1, IC1.24, JP1.1, R5.2, R6.1, R7.1, R8.1, U2.10, U2.16, U4.1, U6.3, U6.8; no longer U$4.#24, U$4.24, U$4.@24
- net VDDA: now also IC1.22; no longer U$4.#22, U$4.22, U$4.@22
Routing:
- net N$10: track 0.00 -> 33.3 mm
- net N$11: track 0.00 -> 26.3 mm
- net N$16: track 0.00 -> 26.2 mm
- net N$17: track 0.00 -> 25.7 mm
- net N$12: track 0.00 -> 25.7 mm
- net VCC: track 0.00 -> 23.4 mm
- net N$9: track 0.00 -> 22.4 mm
- net LATCH: track 0.00 -> 20.9 mm
- net N$8: track 0.00 -> 20.3 mm
- net N$7: track 0.00 -> 18.8 mm
- net CLOCK: track 0.00 -> 18.3 mm
- net N$6: track 0.00 -> 16.1 mm
- net N$4: track 0.00 -> 15.9 mm
- net N$5: track 0.00 -> 12.8 mm
- net N$2: track 0.00 -> 11.2 mm
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- added copper zone on layer 1, net GND
- added copper zone on layer 16, net GND
- added copper zone on layer 1, net TOUCH
Other:
- board size 160 x 134.3 mm -> 88.9 x 105.4 mm
- board text added: "0"
- board text added: "7 Seg"
- board text added: "A0/D0"
- board text added: "A1/D1"
- board text added: "A2/D2"
- board text added: "Based on design by:"
- board text added: "Buzzer"
- board text added: "CLOCK"
- board text added: "Cap Sense"
- board text added: "D2/D9"
- board text added: "D5"
- board text added: "D6"
- board text added: "D7"
- board text added: "Danger Shield 2.0"
- board text added: "GND"
- board text added: "LATCH"
- board text added: "LDR"
- board text added: "Power"
- board text added: "Reset"
- board text added: "SERIAL_OUT"
- board text added: "Sensor"
- board text added: "Shift Reg"
- board text added: "Temp"
- board text added: "VCC"
- board text added: "Zach Hoeken and SparkFun"

Commit message: finished routing
Parts:
- added U$1: (no value), Spark:SPARK_LOGO_PLUS_PLANE
Connections:
- removed net VDDA: IC1.22
- new net VCC3V3: C1.1, IC1.22, R5.2, R6.1, R7.1, R8.1, U4.1
- net VCC: no longer C1.1, R5.2, R6.1, R7.1, R8.1, U4.1
Routing:
- net VCC3V3: track 0.00 -> 172.5 mm
- net VCC: track 23.4 -> 160.5 mm
- net CLOCK: track 18.3 -> 120.8 mm
- net B1: track 0.00 -> 95.7 mm, vias 0 -> 1
- net B3: track 0.00 -> 84.9 mm, vias 0 -> 1
- net B2: track 0.00 -> 84.3 mm, vias 0 -> 1
- net LATCH: track 20.9 -> 98.6 mm
- net S1: track 0.00 -> 76.9 mm
- net SERIAL_IN: track 0.00 -> 75.2 mm
- net TOUCH_S: track 0.00 -> 70.7 mm
- net S2: track 0.00 -> 68.9 mm
- net TOUCH_R: track 0.00 -> 65.7 mm
- net CDS: track 0.00 -> 64.1 mm, vias 0 -> 1
- net TEMP: track 0.00 -> 62.9 mm, vias 0 -> 1
- net S3: track 0.00 -> 57.4 mm
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Other:
- board text added: "A6"
- board text added: "A7"
- board text added: "D19"
- board text added: "Spark Core"
- board text removed: "D2/D9"
- board text removed: "Power"
- board text removed: "Reset"
- board text removed: "Sensor"

Commit message: added headers
Parts:
- added JP2: M09LOCK, SparkFun-Connectors:1X09_LOCK
- moved JP1 17.9 mm to (1.79, 19.1), turned to 270 degrees
- moved U2 3.88 mm to (9.23, 42.5)
- moved C2 2.42 mm to (14.9, 57.4)
Connections:
- new net D18: IC1.4, JP2.7
- net B1: now also JP2.1
- net B2: now also JP2.2
- net B3: now also JP2.3
- net GND: now also JP2.8
- net LED_G: now also JP2.6
- net LED_R: now also JP2.4
- net LED_Y: now also JP2.5
- net VCC: now also JP2.9
Routing:
- net D18: track 0.00 -> 98.1 mm, vias 0 -> 1
- net LED_G: track 44.6 -> 122.6 mm, vias 0 -> 1
- net LED_Y: track 48.6 -> 118.6 mm, vias 0 -> 1
- net LED_R: track 50.6 -> 112.2 mm, vias 0 -> 1
- net B3: track 84.9 -> 136.6 mm
- net B2: track 84.3 -> 118.8 mm
- net SERIAL_OUT: track 10.5 -> 32.0 mm
- net LATCH: track 98.6 -> 119.4 mm, vias 0 -> 1
- net B1: track 95.7 -> 113.7 mm
- net VCC: track 160.5 -> 177.7 mm
- net CLOCK: track 120.8 -> 132.3 mm
- net SERIAL_IN: track 75.2 -> 82.9 mm
- net N$4: track 15.9 -> 23.2 mm
- net N$2: track 11.2 -> 16.6 mm
- net N$8: track 20.3 -> 25.7 mm
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Other:
- board text added: "Based on designs by:"
- board text added: "D0"
- board text added: "D1"
- board text added: "D18"
- board text added: "D2"
- board text added: "Zach Hoeken and Chris Taylor/SparkFun"
- board text removed: "Based on design by:"
- board text removed: "Zach Hoeken and SparkFun"

Commit message: added logo, v1
Parts:
- moved SG1 0.40 mm to (77.5, 55.5)
Routing:
- net BIRD: track 0.00 -> 50.8 mm
- net D18: track 98.1 -> 91.2 mm
- net VCC3V3: track 172.5 -> 171.0 mm
- net LATCH: vias 1 -> 0
- added copper zone on layer 16, net BIRD
Other:
- board text added: "0.1uF"
- board text added: "10pF"
- board text added: "Plover Electric"
- board text added: "Ver 1.0 2014 (CC BY-SA 3.0)"
- board text added: "plover.io/danger"
