File: danger.sch (EAGLE design)
At the start: 7 parts

Commit message: redid based on sparkfun design
Parts:
- removed U$1, U$3: SLIDER, SparkFun-Electromechanical:SLIDER
- removed U$4: SPARK_CORE, Spark:SPARK_CORE
- added C1, C2: 0.1uF, SparkFun-Passives:CAPPTH2
- added C3: 10pF, SparkFun-Passives:CAPPTH2
- added IC1: SPARK_CORECORE, Spark:SPARK_CORECORE
- added JP1: (no value), SparkFun:M05PTH
- added LED1: Red, SparkFun:LED5MM
- added LED2: Yellow, SparkFun:LED5MM
- added LED3: Green, SparkFun:LED5MM
- added R1, R10, R11, R12, R13, R14, R15, R16, R2, R3, R9: 330, SparkFun:RESISTORAXIAL-0.3
- added R17: 1k, SparkFun:RESISTORAXIAL-0.3
- added R30: 10K, SparkFun:RESISTORAXIAL-0.3
- added R4: 10M, SparkFun:RESISTORAXIAL-0.3
- added R5: CdS, SparkFun:PHOTOCELLPTH
- added R6: Slider3, SparkFun:SLIDER
- added R7: Slider2, SparkFun:SLIDER
- added R8: Slider1, SparkFun:SLIDER
- added SG1: BUZZER, SparkFun:BUZZERPTH
- added U2: 74LS595N, SparkFun:74LS595N
- added U4: TMP36, SparkFun-Sensors:TMP36GT9
- added U6: 7-SEGMENT-DISPLAY-1"-RED, SparkFun:7-SEGMENT-DISPLAY-1"-RED
- S1: value (none) -> Button1; device SparkFun-Electromechanical:TAC_SWITCHPTH -> SparkFun:SWITCH-MOMENTARY-212MM
- S2: value (none) -> Button2; device SparkFun-Electromechanical:TAC_SWITCHPTH -> SparkFun:SWITCH-MOMENTARY-212MM
- S3: value (none) -> Button3; device SparkFun-Electromechanical:TAC_SWITCHPTH -> SparkFun:SWITCH-MOMENTARY-212MM
- U$2: value SLIDER -> OSHW-LOGOM; device SparkFun-Electromechanical:SLIDER -> SparkFun-Aesthetics:OSHW-LOGOM
Connections:
- new net B1: IC1.D0, S1.2
- new net B2: IC1.D1, S2.2
- new net B3: IC1.D2, S3.2
- new net BUZZER: IC1.TX, SG1.1
- new net CDS: IC1.A6, R30.2, R5.P$1
- new net CLOCK: IC1.A3, JP1.3, U2.SCK
- new net GND: C1.2, C2.2, C3.2, IC1.GND@2, IC1.GND@21, JP1.5, R1.1, R2.1, R3.1, R30.1, R6.A, R7.A, R8.A, S1.1, S2.1, S3.1, SG1.2, U2.G, U2.GND, U4.GND
- new net LATCH: IC1.A4, JP1.2, U2.RCK
- new net LED_G: IC1.D7, LED3.A
- new net LED_R: IC1.D5, LED1.A
- new net LED_Y: IC1.D6, LED2.A
- new net N$10: R16.1, U2.QH
- new net N$11: R9.2, U6.A
- new net N$12: R10.2, U6.B
- new net N$13: R11.2, U6.C
- new net N$14: R12.2, U6.D
- new net N$15: R13.2, U6.E
- new net N$16: R14.2, U6.F
- new net N$17: R15.2, U6.G
- new net N$18: R16.2, U6.DP
- new net N$19: LED2.C, R2.2
- new net N$2: R9.1, U2.QA
- new net N$20: LED3.C, R3.2
- new net N$3: LED1.C, R1.2
- new net N$4: R10.1, U2.QB
- new net N$5: R11.1, U2.QC
- new net N$6: R12.1, U2.QD
- new net N$7: R13.1, U2.QE
- new net N$8: R14.1, U2.QF
- new net N$9: R15.1, U2.QG
- new net S1: IC1.A0, R8.S
- new net S2: IC1.A1, R7.S
- new net S3: IC1.A2, R6.S
- new net SERIAL_IN: IC1.A5, U2.SER
- new net SERIAL_OUT: JP1.4, U2.QH*
- new net TEMP: IC1.A7, U4.VOUT
- new net TOUCH: C3.1, R17.2, R4.2
- new net TOUCH_R: IC1.D3, R17.1
- new net TOUCH_S: IC1.D4, R4.1
- new net VCC: C1.1, C2.1, IC1.RAW, JP1.1, R5.P$2, R6.E, R7.E, R8.E, U2.SCL, U2.VCC, U4.VCC, U6.G1, U6.G2
Other:
- note added: "Cap Sense"
- note added: "Chris Taylor"
- note added: "Light Sensor"
- note added: "Original design: Zach Hoeken"

Commit message: finished routing
Connections:
- new net VCC3V3: C1.1, IC1.VDDA, R5.P$2, R6.E, R7.E, R8.E, U4.VCC
- net VCC: no longer C1.1, R5.P$2, R6.E, R7.E, R8.E, U4.VCC
Changed lines of the file:
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@@
 <part name="R7" library="SparkFun" deviceset="SLIDER" device="" value="Slider2"/>
 <part name="R6" library="SparkFun" deviceset="SLIDER" device="" value="Slider3"/>
-<part name="P+1" library="SparkFun" deviceset="VCC" device=""/>
-<part name="P+2" library="SparkFun" deviceset="VCC" device=""/>
-<part name="P+3" library="SparkFun" deviceset="VCC" device=""/>
+<part name="P+1" library="SparkFun" deviceset="VCC" device="" value="VCC3v3"/>
+<part name="P+2" library="SparkFun" deviceset="VCC" device="" value="VCC3v3"/>
+<part name="P+3" library="SparkFun" deviceset="VCC" device="" value="VCC3v3"/>
 <part name="GND1" library="SparkFun" deviceset="GND" device=""/>
 <part name="GND2" library="SparkFun" deviceset="GND" device=""/>
@@
 <part name="R5" library="SparkFun" deviceset="PHOTOCELL" device="PTH" value="CdS"/>
 <part name="R30" library="SparkFun" deviceset="RESISTOR" device="AXIAL-0.3" value="10K"/>
-<part name="P+6" library="SparkFun" deviceset="VCC" device=""/>
+<part name="P+6" library="SparkFun" deviceset="VCC" device="" value="VCC3v3"/>
 <part name="GND6" library="SparkFun" deviceset="GND" device=""/>
-<part name="P+7" library="SparkFun" deviceset="VCC" device=""/>
+<part name="P+7" library="SparkFun" deviceset="VCC" device="" value="VCC3v3"/>
 <part name="GND7" library="SparkFun" deviceset="GND" device=""/>
 <part name="U2" library="SparkFun" deviceset="74*595" device="N" technology="LS"/>
@@
 <part name="U4" library="SparkFun-Sensors" deviceset="TMP36" device="GT9" value="TMP36"/>
 <part name="C1" library="SparkFun-Passives" deviceset="CAP" device="PTH2" value="0.1uF"/>
-<part name="P+10" library="SparkFun" deviceset="VCC" device=""/>
+<part name="P+10" library="SparkFun" deviceset="VCC" device="" value="VCC3v3"/>
 <part name="GND8" library="SparkFun" deviceset="GND" device=""/>
 <part name="C2" library="SparkFun-Passives" deviceset="CAP" device="PTH2" value="0.1uF"/>
@@
 <part name="GND19" library="SparkFun" deviceset="GND" device=""/>
 <part name="GND4" library="SparkFun" deviceset="GND" device=""/>
+<part name="P+5" library="SparkFun" deviceset="VCC" device="" value="VCC3v3"/>
 </parts>
 <sheets>
@@
 <instance part="GND19" gate="1" x="121.92" y="106.68"/>
 <instance part="GND4" gate="1" x="55.88" y="114.3"/>
+<instance part="P+5" gate="1" x="111.76" y="116.84"/>
 </instances>
 <busses>
@@
 <nets>
 <net name="VCC" class="0">
-<segment>
-<wire x1="48.26" y1="78.74" x2="48.26" y2="81.28" width="0.1524" layer="91"/>
-<pinref part="R6" gate="G$1" pin="E"/>
-<pinref part="P+1" gate="1" pin="VCC"/>
-</segment>
-<segment>
-<wire x1="33.02" y1="78.74" x2="33.02" y2="81.28" width="0.1524" layer="91"/>
-<pinref part="R7" gate="G$1" pin="E"/>
-<pinref part="P+2" gate="1" pin="VCC"/>
-</segment>
-<segment>
-<wire x1="17.78" y1="78.74" x2="17.78" y2="81.28" width="0.1524" layer="91"/>
-<pinref part="R8" gate="G$1" pin="E"/>
-<pinref part="P+3" gate="1" pin="VCC"/>
-</segment>
-<segment>
-<wire x1="33.02" y1="165.1" x2="33.02" y2="162.56" width="0.1524" layer="91"/>
-<pinref part="R5" gate="G$1" pin="P$2"/>
-<pinref part="P+6" gate="1" pin="VCC"/>
-</segment>
 <segment>
 <wire x1="121.92" y1="160.02" x2="119.38" y2="160.02" width="0.1524" layer="91"/>
@@
 </segment>
 <segment>
-<pinref part="U4" gate="G$1" pin="VCC"/>
-<wire x1="63.5" y1="154.94" x2="60.96" y2="154.94" width="0.1524" layer="91"/>
-<wire x1="60.96" y1="154.94" x2="60.96" y2="157.48" width="0.1524" layer="91"/>
-<pinref part="P+7" gate="1" pin="VCC"/>
-</segment>
-<segment>
-<pinref part="C1" gate="G$1" pin="1"/>
-<pinref part="P+10" gate="1" pin="VCC"/>
-<wire x1="50.8" y1="160.02" x2="50.8" y2="157.48" width="0.1524" layer="91"/>
-</segment>
-<segment>
 <pinref part="C2" gate="G$1" pin="1"/>
 <pinref part="P+11" gate="1" pin="VCC"/>
@@
 <net name="SERIAL_IN" class="0">
 <segment>
-<wire x1="121.92" y1="167.64" x2="104.14" y2="167.64" width="0.1524" layer="91"/>
+<wire x1="121.92" y1="167.64" x2="116.84" y2="167.64" width="0.1524" layer="91"/>
 <pinref part="U2" gate="A" pin="SER"/>
-<label x="104.14" y="167.64" size="1.4224" layer="95" rot="R180" xref="yes"/>
+<label x="116.84" y="167.64" size="1.4224" layer="95" rot="R180" xref="yes"/>
 </segment>
 <segment>
@@
 <net name="CLOCK" class="0">
 <segment>
-<wire x1="121.92" y1="162.56" x2="104.14" y2="162.56" width="0.1524" layer="91"/>
+<wire x1="121.92" y1="162.56" x2="116.84" y2="162.56" width="0.1524" layer="91"/>
 <pinref part="U2" gate="A" pin="SCK"/>
-<label x="104.14" y="162.56" size="1.4224" layer="95" rot="R180" xref="yes"/>
+<label x="116.84" y="162.56" size="1.4224" layer="95" rot="R180" xref="yes"/>
 </segment>
 <segment>
@@
 <net name="LATCH" class="0">
 <segment>
-<wire x1="121.92" y1="154.94" x2="104.14" y2="154.94" width="0.1524" layer="91"/>
+<wire x1="121.92" y1="154.94" x2="116.84" y2="154.94" width="0.1524" layer="91"/>
 <pinref part="U2" gate="A" pin="RCK"/>
-<label x="104.14" y="154.94" size="1.4224" layer="95" rot="R180" xref="yes"/>
+<label x="116.84" y="154.94" size="1.4224" layer="95" rot="R180" xref="yes"/>
 </segment>
 <segment>
@@
 </segment>
 </net>
+<net name="VCC3V3" class="0">
+<segment>
+<pinref part="IC1" gate="G$1" pin="VDDA"/>
+<pinref part="P+5" gate="1" pin="VCC"/>
+<wire x1="106.68" y1="114.3" x2="111.76" y2="114.3" width="0.1524" layer="91"/>
+<wire x1="111.76" y1="114.3" x2="111.76" y2="116.84" width="0.1524" layer="91"/>
+</segment>
+<segment>
+<wire x1="17.78" y1="78.74" x2="17.78" y2="81.28" width="0.1524" layer="91"/>
+<pinref part="R8" gate="G$1" pin="E"/>
+<pinref part="P+3" gate="1" pin="VCC"/>
+</segment>
+<segment>
+<wire x1="33.02" y1="78.74" x2="33.02" y2="81.28" width="0.1524" layer="91"/>
+<pinref part="R7" gate="G$1" pin="E"/>
+<pinref part="P+2" gate="1" pin="VCC"/>
+</segment>
+<segment>
+<wire x1="48.26" y1="78.74" x2="48.26" y2="81.28" width="0.1524" layer="91"/>
+<pinref part="R6" gate="G$1" pin="E"/>
+<pinref part="P+1" gate="1" pin="VCC"/>
+</segment>
+<segment>
+<wire x1="33.02" y1="165.1" x2="33.02" y2="162.56" width="0.1524" layer="91"/>
+<pinref part="R5" gate="G$1" pin="P$2"/>
+<pinref part="P+6" gate="1" pin="VCC"/>
+</segment>
+<segment>
+<pinref part="U4" gate="G$1" pin="VCC"/>
+<wire x1="63.5" y1="154.94" x2="60.96" y2="154.94" width="0.1524" layer="91"/>
+<wire x1="60.96" y1="154.94" x2="60.96" y2="157.48" width="0.1524" layer="91"/>
+<pinref part="P+7" gate="1" pin="VCC"/>
+</segment>
+<segment>
+<pinref part="C1" gate="G$1" pin="1"/>
+<pinref part="P+10" gate="1" pin="VCC"/>
+<wire x1="50.8" y1="160.02" x2="50.8" y2="157.48" width="0.1524" layer="91"/>
+</segment>
+</net>

Commit message: added headers
Parts:
- added JP2: M09LOCK, SparkFun-Connectors:M09LOCK
Connections:
- new net D18: IC1.RX, JP2.7
- net B1: now also JP2.1
- net B2: now also JP2.2
- net B3: now also JP2.3
- net GND: now also JP2.8
- net LED_G: now also JP2.6
- net LED_R: now also JP2.4
- net LED_Y: now also JP2.5
- net VCC: now also JP2.9
Changed lines of the file:
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@@
 <layer number="54" name="bGND_GNDA" color="1" fill="9" visible="no" active="no"/>
 <layer number="56" name="wert" color="7" fill="1" visible="no" active="no"/>
+<layer number="57" name="tCAD" color="7" fill="1" visible="no" active="no"/>
 <layer number="91" name="Nets" color="2" fill="1" visible="yes" active="yes"/>
 <layer number="92" name="Busses" color="1" fill="1" visible="yes" active="yes"/>
@@
 <layer number="97" name="Info" color="7" fill="1" visible="yes" active="yes"/>
 <layer number="98" name="Guide" color="6" fill="1" visible="yes" active="yes"/>
+<layer number="99" name="SpiceOrder" color="7" fill="1" visible="yes" active="yes"/>
 <layer number="100" name="Muster" color="7" fill="1" visible="no" active="no"/>
 <layer number="101" name="Patch_Top" color="12" fill="4" visible="yes" active="yes"/>
@@
 <layer number="111" name="LPC17xx" color="7" fill="1" visible="yes" active="yes"/>
 <layer number="112" name="tSilk" color="7" fill="1" visible="yes" active="yes"/>
+<layer number="113" name="IDFDebug" color="4" fill="1" visible="yes" active="yes"/>
 <layer number="116" name="Patch_BOT" color="9" fill="4" visible="yes" active="yes"/>
 <layer number="121" name="_tsilk" color="7" fill="1" visible="yes" active="yes"/>
@@
 <layer number="132" name="bAdjust" color="7" fill="1" visible="yes" active="yes"/>
 <layer number="144" name="Drill_legend" color="7" fill="1" visible="yes" active="yes"/>
+<layer number="150" name="Notes" color="7" fill="1" visible="yes" active="yes"/>
 <layer number="151" name="HeatSink" color="7" fill="1" visible="yes" active="yes"/>
 <layer number="152" name="_bDocu" color="7" fill="1" visible="yes" active="yes"/>
+<layer number="153" name="FabDoc1" color="7" fill="1" visible="yes" active="yes"/>
+<layer number="154" name="FabDoc2" color="7" fill="1" visible="yes" active="yes"/>
+<layer number="155" name="FabDoc3" color="7" fill="1" visible="yes" active="yes"/>
 <layer number="199" name="Contour" color="7" fill="1" visible="yes" active="yes"/>
 <layer number="200" name="200bmp" color="1" fill="10" visible="yes" active="yes"/>
@@
 <part name="GND4" library="SparkFun" deviceset="GND" device=""/>
 <part name="P+5" library="SparkFun" deviceset="VCC" device="" value="VCC3v3"/>
+<part name="JP2" library="SparkFun-Connectors" deviceset="M09" device="LOCK"/>
+<part name="P+14" library="SparkFun" deviceset="VCC" device=""/>
+<part name="GND20" library="SparkFun" deviceset="GND" device=""/>
 </parts>
 <sheets>
@@
 <instance part="GND4" gate="1" x="55.88" y="114.3"/>
 <instance part="P+5" gate="1" x="111.76" y="116.84"/>
+<instance part="JP2" gate="G$1" x="66.04" y="22.86"/>
+<instance part="P+14" gate="1" x="78.74" y="35.56"/>
+<instance part="GND20" gate="1" x="91.44" y="27.94"/>
 </instances>
 <busses>
@@
 <wire x1="68.58" y1="124.46" x2="68.58" y2="129.54" width="0.1524" layer="91"/>
 </segment>
+<segment>
+<pinref part="JP2" gate="G$1" pin="9"/>
+<pinref part="P+14" gate="1" pin="VCC"/>
+<wire x1="76.2" y1="33.02" x2="78.74" y2="33.02" width="0.1524" layer="91"/>
+<wire x1="78.74" y1="33.02" x2="78.74" y2="35.56" width="0.1524" layer="91"/>
+</segment>
 </net>
 <net name="GND" class="0">
@@
 <wire x1="55.88" y1="119.38" x2="55.88" y2="116.84" width="0.1524" layer="91"/>
 </segment>
+<segment>
+<pinref part="JP2" gate="G$1" pin="8"/>
+<pinref part="GND20" gate="1" pin="GND"/>
+<wire x1="76.2" y1="30.48" x2="91.44" y2="30.48" width="0.1524" layer="91"/>
+</segment>
 </net>
 <net name="N$3" class="0">
@@
 <label x="109.22" y="78.74" size="1.4224" layer="95" xref="yes"/>
 </segment>
+<segment>
+<pinref part="JP2" gate="G$1" pin="3"/>
+<wire x1="76.2" y1="17.78" x2="78.74" y2="17.78" width="0.1524" layer="91"/>
+<label x="78.74" y="17.78" size="1.4224" layer="95" xref="yes"/>
+</segment>
 </net>
 <net name="B2" class="0">
@@
 <label x="109.22" y="73.66" size="1.4224" layer="95" xref="yes"/>
 </segment>
+<segment>
+<pinref part="JP2" gate="G$1" pin="2"/>
+<wire x1="76.2" y1="15.24" x2="78.74" y2="15.24" width="0.1524" layer="91"/>
+<label x="78.74" y="15.24" size="1.4224" layer="95" xref="yes"/>
+</segment>
 </net>
 <net name="B1" class="0">
@@
 <wire x1="106.68" y1="68.58" x2="109.22" y2="68.58" width="0.1524" layer="91"/>
 <label x="109.22" y="68.58" size="1.4224" layer="95" xref="yes"/>
+</segment>
+<segment>
+<pinref part="JP2" gate="G$1" pin="1"/>
+<wire x1="76.2" y1="12.7" x2="78.74" y2="12.7" width="0.1524" layer="91"/>
+<label x="78.74" y="12.7" size="1.4224" layer="95" xref="yes"/>
 </segment>
 </net>
@@
 <label x="109.22" y="93.98" size="1.4224" layer="95" xref="yes"/>
 </segment>
+<segment>
+<pinref part="JP2" gate="G$1" pin="4"/>
+<wire x1="76.2" y1="20.32" x2="78.74" y2="20.32" width="0.1524" layer="91"/>
+<label x="78.74" y="20.32" size="1.4224" layer="95" xref="yes"/>
+</segment>
 </net>
 <net name="LED_G" class="0">
@@
 <label x="109.22" y="104.14" size="1.4224" layer="95" xref="yes"/>
 </segment>
+<segment>
+<pinref part="JP2" gate="G$1" pin="6"/>
+<wire x1="76.2" y1="25.4" x2="78.74" y2="25.4" width="0.1524" layer="91"/>
+<label x="78.74" y="25.4" size="1.4224" layer="95" xref="yes"/>
+</segment>
 </net>
 <net name="LED_Y" class="0">
@@
 <wire x1="106.68" y1="99.06" x2="109.22" y2="99.06" width="0.1524" layer="91"/>
 <label x="109.22" y="99.06" size="1.4224" layer="95" xref="yes"/>
+</segment>
+<segment>
+<pinref part="JP2" gate="G$1" pin="5"/>
+<wire x1="76.2" y1="22.86" x2="78.74" y2="22.86" width="0.1524" layer="91"/>
+<label x="78.74" y="22.86" size="1.4224" layer="95" xref="yes"/>
 </segment>
 </net>
@@
 </segment>
 </net>
+<net name="D18" class="0">
+<segment>
+<pinref part="IC1" gate="G$1" pin="RX"/>
+<wire x1="68.58" y1="109.22" x2="71.12" y2="109.22" width="0.1524" layer="91"/>
+<label x="68.58" y="109.22" size="1.4224" layer="95" rot="R180" xref="yes"/>
+</segment>
+<segment>
+<pinref part="JP2" gate="G$1" pin="7"/>
+<wire x1="76.2" y1="27.94" x2="78.74" y2="27.94" width="0.1524" layer="91"/>
+<label x="78.74" y="27.94" size="1.4224" layer="95" xref="yes"/>
+</segment>
+</net>
